File: Bendy1.brd (EAGLE design)
At the start: 8 parts, among them J1 Qwiic Right Angle, U1 MTCH6301-I/PT

Commit message: Initial commit
Routing:
- net GND: track 0.00 -> 3.91 mm
- net TX5: track 147.4 -> 148.7 mm
- net +3V3: track 13.3 -> 14.5 mm, vias 3 -> 5
Other:
- board outline added: 186.2 x 93.3 mm
Changed lines of the file:
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@@
 <drawing>
 <settings>
-<setting alwaysvectorfont="no"/>
+<setting alwaysvectorfont="yes"/>
 <setting verticaltext="up"/>
 </settings>
-<grid distance="10" unitdist="mil" unit="mil" style="lines" multiple="1" display="no" altdistance="5" altunitdist="mil" altunit="mil"/>
+<grid distance="5" unitdist="mil" unit="mil" style="lines" multiple="1" display="no" altdistance="5" altunitdist="mil" altunit="mil"/>
 <layers>
 <layer number="1" name="Top" color="4" fill="1" visible="yes" active="yes"/>
@@
 </layers>
 <board>
+<fusionsync huburn="a.YnVzaW5lc3M6c3Z2c2QzNA" projecturn="a.YnVzaW5lc3M6c3Z2c2QzNCMyMDIxMDQxNTQwMzQ3MTYzMQ" f3durn="urn:adsk.wipprod:dm.lineage:uzEAV6WZRViNt0AiRt7dWQ" pcbguid="" lastpulledtime="" lastsyncedchangeguid="" latestrevisionid="3742b59a-0cc7-4492-a824-a101a1e10ba2" lastsyncedrevisionid="3742b59a-0cc7-4492-a824-a101a1e10ba2" lastboardhashguid="4435e586-4238-db4c-d6ba-827551b01d8d" lastpushedtime="2024-04-04T15:45:10Z" linktopcb3d="true"/>
 <plain>
 <dimension x1="67.31" y1="25.08" x2="57.31" y2="25.08" x3="62.31" y3="25.08" textsize="1.778" layer="51" extlength="5"/>
@@
 <dimension x1="0" y1="24.13" x2="-65.913" y2="25.019" x3="-32.9565" y3="21.971" textsize="1.778" layer="51" dtype="horizontal"/>
 <wire x1="-66.04" y1="25.4" x2="-66.04" y2="85.09" width="0.4064" layer="51"/>
+<wire x1="-0.889" y1="33.02" x2="-0.889" y2="-0.635" width="0" layer="20"/>
+<wire x1="-0.889" y1="-0.635" x2="22.86" y2="-0.635" width="0" layer="20"/>
+<wire x1="-0.889" y1="33.02" x2="-66.548" y2="33.02" width="0" layer="20"/>
+<wire x1="-66.548" y1="33.02" x2="-67.818" y2="34.29" width="0" layer="20"/>
+<wire x1="-67.818" y1="34.29" x2="-67.818" y2="84.582" width="0" layer="20"/>
+<wire x1="-67.818" y1="84.582" x2="-66.421" y2="85.979" width="0" layer="20"/>
+<wire x1="-66.421" y1="85.979" x2="1.016" y2="85.852" width="0" layer="20"/>
+<wire x1="1.016" y1="85.852" x2="19.05" y2="67.818" width="0" layer="20"/>
+<wire x1="19.05" y1="67.818" x2="19.05" y2="32.766" width="0" layer="20"/>
+<wire x1="19.05" y1="32.766" x2="29.337" y2="22.86" width="0" layer="20"/>
+<wire x1="29.337" y1="22.86" x2="62.992" y2="22.86" width="0" layer="20"/>
+<wire x1="62.992" y1="22.86" x2="64.77" y2="24.638" width="0" layer="20"/>
+<wire x1="64.77" y1="24.638" x2="64.77" y2="92.075" width="0" layer="20"/>
+<wire x1="64.77" y1="92.075" x2="65.405" y2="92.71" width="0" layer="20"/>
+<wire x1="65.405" y1="92.71" x2="117.348" y2="92.71" width="0" layer="20"/>
+<wire x1="117.348" y1="92.71" x2="118.364" y2="91.694" width="0" layer="20"/>
+<wire x1="118.364" y1="91.694" x2="118.364" y2="24.765" width="0" layer="20"/>
+<wire x1="118.364" y1="24.765" x2="110.871" y2="17.272" width="0" layer="20"/>
+<wire x1="110.871" y1="17.272" x2="30.607" y2="17.272" width="0" layer="20"/>
+<wire x1="30.607" y1="17.272" x2="26.035" y2="12.446" width="0" layer="20"/>
+<wire x1="26.035" y1="12.446" x2="23.495" y2="12.446" width="0" layer="20"/>
+<wire x1="23.495" y1="12.446" x2="22.86" y2="11.811" width="0" layer="20"/>
+<wire x1="22.86" y1="11.811" x2="22.86" y2="-0.635" width="0" layer="20"/>
 </plain>
 <attributes>
@@
 </class>
 </classes>
-<designrules name="default">
+<designrules name="default *">
 <description language="de">&lt;b&gt;EAGLE Design Rules&lt;/b&gt;
 &lt;p&gt;
@@
 design rules under a new name.</description>
 <param name="layerSetup" value="(1*16)"/>
-<param name="mtCopper" value="0.035mm 0.035mm 0.035mm 0.035mm 0.035mm 0.035mm 0.035mm 0.035mm 0.035mm 0.035mm 0.035mm 0.035mm 0.035mm 0.035mm 0.035mm 0.035mm"/>
-<param name="mtIsolate" value="1.5mm 0.15mm 0.2mm 0.15mm 0.2mm 0.15mm 0.2mm 0.15mm 0.2mm 0.15mm 0.2mm 0.15mm 0.2mm 0.15mm 0.2mm"/>
+<param name="mtCopper" value="0.018mm 0.035mm 0.035mm 0.035mm 0.035mm 0.035mm 0.035mm 0.035mm 0.035mm 0.035mm 0.035mm 0.035mm 0.035mm 0.035mm 0.035mm 0.018mm"/>
+<param name="mtIsolate" value="0.1mm 0.15mm 0.2mm 0.15mm 0.2mm 0.15mm 0.2mm 0.15mm 0.2mm 0.15mm 0.2mm 0.15mm 0.2mm 0.15mm 0.2mm"/>
 <param name="mdWireWire" value="6mil"/>
 <param name="mdWirePad" value="6mil"/>
@@
 <contactref element="U1" pad="29"/>
 <contactref element="C4" pad="1"/>
-<polygon width="0.1524" layer="1">
-<vertex x="0" y="23.495"/>
-<vertex x="0" y="0"/>
-<vertex x="22.86" y="0"/>
-<vertex x="22.86" y="24.13"/>
-<vertex x="0" y="24.13"/>
+<wire x1="16.1035875" y1="15.96495625" x2="18.639875" y2="18.50124375" width="0.4064" layer="1"/>
+<wire x1="18.639875" y1="18.50124375" x2="18.639875" y2="18.825121875" width="0.4064" layer="1"/>
+<polygon width="0.4064" layer="1">
+<vertex x="-0.889" y="-0.635"/>
+<vertex x="-0.889" y="24.13"/>
+<vertex x="15.24" y="24.13"/>
+<vertex x="22.86" y="16.51"/>
+<vertex x="22.86" y="-0.635"/>
 </polygon>
 </signal>
@@
 <contactref element="U1" pad="28"/>
 <contactref element="C4" pad="2"/>
-<wire x1="7.586040625" y1="17.746040625" x2="7.586040625" y2="16.54395625" width="0.1524" layer="1"/>
-<wire x1="7.586040625" y1="16.54395625" x2="8.730725" y2="15.399271875" width="0.1524" layer="1"/>
-<wire x1="16.669271875" y1="15.399271875" x2="18.0975" y2="16.8275" width="0.1524" layer="1"/>
-<wire x1="18.0975" y1="16.8275" x2="19.274875" y2="18.004875" width="0.1524" layer="1"/>
-<wire x1="19.274875" y1="18.004875" x2="19.460121875" y2="18.004875" width="0.1524" layer="1"/>
 <polygon width="0.1524" layer="16">
-<vertex x="0" y="24.13"/>
-<vertex x="22.86" y="24.13"/>
-<vertex x="22.86" y="0"/>
-<vertex x="0" y="0"/>
+<vertex x="-0.889" y="-0.635"/>
+<vertex x="-0.889" y="24.13"/>
+<vertex x="15.24" y="24.13"/>
+<vertex x="22.86" y="16.51"/>
+<vertex x="22.86" y="-0.635"/>
 </polygon>
-<wire x1="17.995" y1="3.81" x2="19.29895625" y2="5.11395625" width="0.1524" layer="1"/>
-<wire x1="19.29895625" y1="5.11395625" x2="19.651040625" y2="5.11395625" width="0.1524" layer="1"/>
-<via x="6.35" y="3.81" extent="1-16" drill="0.3"/>
-<wire x1="5.08" y1="4.31" x2="5.85" y2="4.31" width="0.1524" layer="1"/>
-<wire x1="5.85" y1="4.31" x2="6.35" y2="3.81" width="0.1524" layer="1"/>
-<wire x1="7.586040625" y1="17.746040625" x2="8.89" y2="19.05" width="0.1524" layer="1"/>
-<via x="8.89" y="19.05" extent="1-16" drill="0.35"/>
-<wire x1="18.0975" y1="16.8275" x2="17.78" y2="17.145" width="0.1524" layer="1"/>
-<wire x1="17.78" y1="17.145" x2="17.145" y2="17.145" width="0.1524" layer="1"/>
-<via x="17.145" y="17.145" extent="1-16" drill="0.35"/>
-<wire x1="19.651040625" y1="5.11395625" x2="16.669271875" y2="7.460725" width="0" layer="19" extent="1-1"/>
-<wire x1="16.669271875" y1="15.399271875" x2="16.669271875" y2="7.460725" width="0" layer="19" extent="1-1"/>
+<wire x1="5.08" y1="4.31" x2="5.723" y2="4.31" width="0.4064" layer="1"/>
+<wire x1="5.723" y1="4.31" x2="6.35" y2="3.683" width="0.4064" layer="1"/>
+<via x="6.35" y="3.683" extent="1-16" drill="0.35"/>
+<wire x1="16.669271875" y1="15.399271875" x2="17.907" y2="16.637" width="0.4064" layer="1"/>
+<via x="17.907" y="16.637" extent="1-16" drill="0.35"/>
+<wire x1="17.907" y1="16.637" x2="19.274875" y2="18.004875" width="0.4064" layer="1"/>
+<wire x1="19.274875" y1="18.004875" x2="19.460121875" y2="18.004875" width="0.4064" layer="1"/>
+<wire x1="17.995" y1="3.81" x2="18.5225" y2="4.3375" width="0.4064" layer="1"/>
+<wire x1="18.5225" y1="4.3375" x2="19.29895625" y2="5.11395625" width="0.4064" layer="1"/>
+<wire x1="19.29895625" y1="5.11395625" x2="19.651040625" y2="5.11395625" width="0.4064" layer="1"/>
+<via x="17.145" y="5.461" extent="1-16" drill="0.35"/>
+<wire x1="17.15964375" y1="6.406496875" x2="17.145" y2="6.391853125" width="0.4064" layer="1"/>
+<wire x1="17.145" y1="6.391853125" x2="17.145" y2="5.461" width="0.4064" layer="1"/>
+<wire x1="16.669271875" y1="7.460725" x2="17.15964375" y2="6.970353125" width="0.4064" layer="1"/>
+<wire x1="17.15964375" y1="6.970353125" x2="17.15964375" y2="6.406496875" width="0.4064" layer="1"/>
+<via x="17.145" y="5.461" extent="1-16" drill="0.35"/>
+<wire x1="17.145" y1="5.461" x2="18.2685" y2="4.3375" width="0.4064" layer="1"/>
+<wire x1="18.2685" y1="4.3375" x2="18.5225" y2="4.3375" width="0.4064" layer="1"/>
+<wire x1="7.586040625" y1="17.746040625" x2="8.255" y2="17.07708125" width="0.4064" layer="1"/>
+<wire x1="8.255" y1="17.07708125" x2="8.255" y2="16.891" width="0.4064" layer="1"/>
+<via x="8.255" y="16.891" extent="1-16" drill="0.35"/>
+<wire x1="8.255" y1="16.891" x2="8.255" y2="16.46815" width="0.4064" layer="1"/>
+<wire x1="8.255" y1="16.46815" x2="8.240353125" y2="16.453503125" width="0.4064" layer="1"/>
+<wire x1="8.240353125" y1="16.453503125" x2="8.240353125" y2="15.88964375" width="0.4064" layer="1"/>
+<wire x1="8.240353125" y1="15.88964375" x2="8.730725" y2="15.399271875" width="0.4064" layer="1"/>
 </signal>
 <signal name="N$2">
@@
 <wire x1="13.989825" y1="16.51" x2="17.495875" y2="20.01605" width="0.4064" layer="16"/>
 <wire x1="17.78" y1="20.32" x2="17.78" y2="67.31" width="0.4064" layer="1"/>
-<wire x1="0.508" y1="84.582" x2="-64.77" y2="84.582" width="0.4064" layer="1"/>
+<wire x1="0.508" y1="84.582" x2="-66.04" y2="84.582" width="0.4064" layer="1"/>
 <wire x1="17.78" y1="67.31" x2="0.508" y2="84.582" width="0.4064" layer="1"/>
 </signal>
@@
 </signals>
 <mfgpreviewcolors>
-<mfgpreviewcolor name="soldermaskcolor" color="0xC8008000"/>
+<mfgpreviewcolor name="soldermaskcolor" color="0xC8CFD138"/>
 <mfgpreviewcolor name="silkscreencolor" color="0xFFFEFEFE"/>
 <mfgpreviewcolor name="backgroundcolor" color="0xFF282828"/>
@@
 </note>
 <note version="8.3" severity="warning">
+Since Version 8.3, EAGLE supports Fusion synchronisation.
+This feature will not be available in this version and saving
+the document will break the link to the Fusion PCB feature.
+</note>
+<note version="8.3" severity="warning">
