File: Bendy1.sch (EAGLE design)
At the start: 8 parts, among them J1 Qwiic Right Angle, U1 MTCH6301-I/PT

Commit message: Initial commit
Other:
- moved on the sheet: J1, J2
Changed lines of the file:
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@@
 <attribute name="VALUE" x="129.2606" y="85.3186" size="2.0828" layer="96" ratio="6" rot="SR0"/>
 </instance>
-<instance part="J1" gate="G$1" x="35.56" y="15.24" smashed="yes">
-<attribute name="VALUE" x="30.48" y="9.906" size="1.778" layer="96" font="vector" align="top-left"/>
-<attribute name="NAME" x="30.48" y="23.114" size="1.778" layer="95" font="vector"/>
-</instance>
-<instance part="GND1" gate="1" x="48.26" y="12.7" smashed="yes" rot="R90">
-<attribute name="VALUE" x="50.8" y="10.16" size="1.778" layer="96" rot="R90"/>
+<instance part="J1" gate="G$1" x="60.96" y="53.34" smashed="yes">
+<attribute name="VALUE" x="55.88" y="48.006" size="1.778" layer="96" font="vector" align="top-left"/>
+<attribute name="NAME" x="55.88" y="61.214" size="1.778" layer="95" font="vector"/>
+</instance>
+<instance part="GND1" gate="1" x="73.66" y="50.8" smashed="yes" rot="R90">
+<attribute name="VALUE" x="76.2" y="48.26" size="1.778" layer="96" rot="R90"/>
 </instance>
 <instance part="GND2" gate="1" x="86.36" y="40.64" smashed="yes" rot="R270">
@@
 <attribute name="VALUE" x="101.6" y="33.02" size="1.778" layer="96" rot="R270"/>
 </instance>
-<instance part="+3V3" gate="G$1" x="53.34" y="15.24" smashed="yes" rot="R270">
-<attribute name="VALUE" x="53.34" y="15.24" size="1.778" layer="96"/>
+<instance part="+3V3" gate="G$1" x="78.74" y="53.34" smashed="yes" rot="R270">
+<attribute name="VALUE" x="78.74" y="53.34" size="1.778" layer="96"/>
 </instance>
 <instance part="GND3" gate="1" x="96.52" y="66.04" smashed="yes" rot="R270">
@@
 <attribute name="VALUE" x="172.72" y="71.12" size="1.778" layer="96" rot="R90"/>
 </instance>
-<instance part="J2" gate="J1" x="38.1" y="63.5" smashed="yes">
-<attribute name="VALUE" x="33.02" y="53.594" size="1.778" layer="96" font="vector"/>
-<attribute name="NAME" x="33.02" y="74.168" size="1.778" layer="95" font="vector"/>
-</instance>
-<instance part="GND5" gate="1" x="48.26" y="58.42" smashed="yes" rot="R90">
-<attribute name="VALUE" x="50.8" y="55.88" size="1.778" layer="96" rot="R90"/>
-</instance>
-<instance part="+3V4" gate="G$1" x="55.88" y="60.96" smashed="yes" rot="R270">
-<attribute name="VALUE" x="55.88" y="60.96" size="1.778" layer="96"/>
+<instance part="J2" gate="J1" x="60.96" y="78.74" smashed="yes">
+<attribute name="VALUE" x="55.88" y="68.834" size="1.778" layer="96" font="vector"/>
+<attribute name="NAME" x="55.88" y="89.408" size="1.778" layer="95" font="vector"/>
+</instance>
+<instance part="GND5" gate="1" x="71.12" y="73.66" smashed="yes" rot="R90">
+<attribute name="VALUE" x="73.66" y="71.12" size="1.778" layer="96" rot="R90"/>
+</instance>
+<instance part="+3V4" gate="G$1" x="78.74" y="76.2" smashed="yes" rot="R270">
+<attribute name="VALUE" x="78.74" y="76.2" size="1.778" layer="96"/>
 </instance>
 <instance part="+3V5" gate="G$1" x="182.88" y="38.1" smashed="yes" rot="R270">
@@
 <segment>
 <pinref part="J1" gate="G$1" pin="3"/>
-<wire x1="43.18" y1="17.78" x2="53.34" y2="17.78" width="0.1524" layer="91"/>
-<label x="53.34" y="17.78" size="1.778" layer="95" rot="MR0"/>
+<wire x1="68.58" y1="55.88" x2="78.74" y2="55.88" width="0.1524" layer="91"/>
+<label x="78.74" y="55.88" size="1.778" layer="95" rot="MR0"/>
 </segment>
 <segment>
 <pinref part="J2" gate="J1" pin="4"/>
-<wire x1="43.18" y1="66.04" x2="58.42" y2="66.04" width="0.1524" layer="91"/>
-<label x="58.42" y="66.04" size="1.778" layer="95" rot="MR0"/>
+<wire x1="66.04" y1="81.28" x2="81.28" y2="81.28" width="0.1524" layer="91"/>
+<label x="81.28" y="81.28" size="1.778" layer="95" rot="MR0"/>
 </segment>
 </net>
@@
 <segment>
 <pinref part="J1" gate="G$1" pin="4"/>
-<wire x1="43.18" y1="20.32" x2="53.34" y2="20.32" width="0.1524" layer="91"/>
-<label x="53.34" y="20.32" size="1.778" layer="95" rot="MR0"/>
+<wire x1="68.58" y1="58.42" x2="78.74" y2="58.42" width="0.1524" layer="91"/>
+<label x="78.74" y="58.42" size="1.778" layer="95" rot="MR0"/>
 </segment>
 <segment>
 <pinref part="J2" gate="J1" pin="3"/>
-<wire x1="43.18" y1="63.5" x2="58.42" y2="63.5" width="0.1524" layer="91"/>
-<label x="58.42" y="63.5" size="1.778" layer="95" rot="MR0"/>
+<wire x1="66.04" y1="78.74" x2="81.28" y2="78.74" width="0.1524" layer="91"/>
+<label x="81.28" y="78.74" size="1.778" layer="95" rot="MR0"/>
 </segment>
 </net>
@@
 <pinref part="J1" gate="G$1" pin="1"/>
 <pinref part="GND1" gate="1" pin="GND"/>
-<wire x1="43.18" y1="12.7" x2="45.72" y2="12.7" width="0.1524" layer="91"/>
+<wire x1="68.58" y1="50.8" x2="71.12" y2="50.8" width="0.1524" layer="91"/>
 </segment>
 <segment>
@@
 <pinref part="J2" gate="J1" pin="1"/>
 <pinref part="GND5" gate="1" pin="GND"/>
-<wire x1="43.18" y1="58.42" x2="45.72" y2="58.42" width="0.1524" layer="91"/>
+<wire x1="66.04" y1="73.66" x2="68.58" y2="73.66" width="0.1524" layer="91"/>
 </segment>
 <segment>
@@
 <pinref part="J1" gate="G$1" pin="2"/>
 <pinref part="+3V3" gate="G$1" pin="+3V3"/>
-<wire x1="43.18" y1="15.24" x2="50.8" y2="15.24" width="0.1524" layer="91"/>
+<wire x1="68.58" y1="53.34" x2="76.2" y2="53.34" width="0.1524" layer="91"/>
 </segment>
 <segment>
@@
 <pinref part="J2" gate="J1" pin="2"/>
 <pinref part="+3V4" gate="G$1" pin="+3V3"/>
-<wire x1="43.18" y1="60.96" x2="53.34" y2="60.96" width="0.1524" layer="91"/>
+<wire x1="66.04" y1="76.2" x2="76.2" y2="76.2" width="0.1524" layer="91"/>
 </segment>
 <segment>
@@
 <segment>
 <pinref part="J2" gate="J1" pin="6"/>
-<wire x1="43.18" y1="71.12" x2="58.42" y2="71.12" width="0.1524" layer="91"/>
-<label x="58.42" y="71.12" size="1.778" layer="95" rot="MR0"/>
+<wire x1="66.04" y1="86.36" x2="81.28" y2="86.36" width="0.1524" layer="91"/>
+<label x="81.28" y="86.36" size="1.778" layer="95" rot="MR0"/>
 </segment>
 </net>
@@
 <segment>
 <pinref part="J2" gate="J1" pin="5"/>
-<wire x1="43.18" y1="68.58" x2="58.42" y2="68.58" width="0.1524" layer="91"/>
-<label x="58.42" y="68.58" size="1.778" layer="95" rot="MR0"/>
-</segment>
-<segment>
+<wire x1="66.04" y1="83.82" x2="81.28" y2="83.82" width="0.1524" layer="91"/>
+<label x="81.28" y="83.82" size="1.778" layer="95" rot="MR0"/>
+</segment>
+<segment>
